File: enkaz-dinleme/enkaz-dinleme-kicad/Enkaz.kicad_pcb (KiCad board)
At the start: 2 copper layers, 30 parts, among them U1 AD8552M_TR, U2 PJ-320D, U3 BH-AAA-B5AK001, U4 AO3401A, U5 XL-1606SURC, Y1 Crystal

Commit message: 3d models add, rough layout
Parts:
- moved P2 84.2 mm to (111.8, 22.9)
- moved P1 78.8 mm to (104.1, 22.9)
- moved C8 74.6 mm to (122.6, 33.0), turned to 180 degrees
- moved C9 70.7 mm to (122.8, 25.4), turned to 180 degrees
- moved C10 70.7 mm to (122.8, 27.9), turned to 180 degrees
- moved U1 57.5 mm to (128.7, 30.5)
- moved C11 57.4 mm to (122.8, 30.5), turned to 180 degrees
- moved C4 33.1 mm to (115.7, 79.8), turned to -90 degrees
- moved C5 30.7 mm to (112.7, 79.8), turned to -90 degrees
- moved PR1 30.7 mm to (146.6, 88.0)
- moved R1 30.7 mm to (132.1, 81.3)
- moved R2 30.7 mm to (132.1, 83.8)
- moved R4 30.7 mm to (132.1, 86.3)
- moved R5 30.7 mm to (132.1, 88.8)
- moved C1 30.7 mm to (127.7, 78.8)
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